File: Geiger-Muller/Geiger-Muller.kicad_pcb (KiCad board)
At the start: 2 copper layers, 105.5 x 55 mm, 24 parts, among them Q1 2N3904, Q2 MPSA42, U1 NE555P, U2 L7805

Commit message: pcb update
Parts:
- added J1: Conn_01x01_Pin, Connector_Wire:SolderWire-1sqmm_1x01_D1.4mm_OD3.9mm, F.Cu at (41.5, 78.5)
- added J2: Conn_01x01_Pin, Connector_Wire:SolderWire-1sqmm_1x01_D1.4mm_OD3.9mm, F.Cu at (135.0, 101.0)
- added J3: Conn_01x01_Pin, Connector_Wire:SolderWire-1sqmm_1x01_D1.4mm_OD3.9mm, F.Cu at (41.5, 84.5)
- added J4: Conn_01x01_Pin, Connector_Wire:SolderWire-1sqmm_1x01_D1.4mm_OD3.9mm, F.Cu at (135.0, 94.0)
Connections:
- R7 pad 2: unconnected-(R7-Pad2) -> Net-(J2-Pin_1)
Routing:
- net Net-(J2-Pin_1): track 0.00 -> 15.0 mm
- net unconnected-(R7-Pad2): track 13.7 -> 0.00 mm, vias 1 -> 0
- net +5V: track 10.1 -> 11.6 mm, vias 1 -> 0
- net Net-(Q1-B): track 30.1 -> 31.2 mm
- net GND: vias 2 -> 0
