File: Geiger-Muller/Geiger-Muller.kicad_sch (KiCad schematic)
At the start: 24 parts, among them Q1 2N3904, Q2 MPSA42, U1 NE555P, U2 L7805

Commit message: pcb update
Parts:
- added J1, J2, J3, J4: Conn_01x01_Pin, Connector_Wire:SolderWire-1sqmm_1x01_D1.4mm_OD3.9mm, symbol Connector:Conn_01x01_Pin
Connections:
- net +5V: now also J1.1 (Pin_1)
- net GND: now also J3.1 (Pin_1), J4.1 (Pin_1)
- net at R7.2: now also J2.1 (Pin_1)
